Commit message: Adjustment to CEMIRA CogArch

File: yumi_description/urdf/yumi.urdf.xacro (robot description, xacro)
@@ -2,26 +2,150 @@
 <robot name="yumi" xmlns:xacro="http://www.ros.org/wiki/xacro">
   <!-- Import Rviz colors -->
-  <xacro:include filename="$(find yumi_description)/urdf/materials.xacro" />
+  <xacro:include filename="$(find yumi_description)/urdf/Util/materials.xacro" />
   <!-- Import utilities -->
-  <xacro:include filename="$(find yumi_description)/urdf/utilities.xacro" />
+  <xacro:include filename="$(find yumi_description)/urdf/Util/utilities.xacro" />
   <!--Import the yumi macro -->
   <xacro:include filename="$(find yumi_description)/urdf/yumi.xacro"/>
   <!--Import the yumi servo gripper macro -->
-  <xacro:include filename="$(find yumi_description)/urdf/yumi_servo_gripper.xacro"/>
- <!-- Import Gazebo plugins -->
-  <xacro:include filename="$(find yumi_description)/gazebo/gazebo.urdf.xacro"/>
-  <!-- Fix to world just for testing -->
-  <link name="world"/>
+  <xacro:include filename="$(find yumi_description)/urdf/Grippers/yumi_servo_gripper.xacro"/>
+  <!-- Import Gazebo plugins -->
+  <xacro:include filename="$(find yumi_description)/urdf/Gazebo/gazebo.urdf.xacro"/>
   <!--yumi-->
-  <xacro:yumi name="yumi" hardware_interface="$(arg prefix)" parent="world">
+  <xacro:yumi name="yumi" hardware_interface="hardware_interface/VelocityJointInterface" parent="${yumi_parent}" >
     <origin xyz="0 0 0.1" rpy="0 0 0" />
   </xacro:yumi>
   <!--right gripper-->
-  <xacro:yumi_servo_gripper name="gripper_r" hardware_interface="$(arg prefix)" parent="yumi_link_7_r">
+  <xacro:yumi_servo_gripper name="gripper_r" hardware_interface="hardware_interface/EffortJointInterface" parent="yumi_link_7_r">
     <origin xyz="0 0 0.007" rpy="0 0 ${PI}" />
   </xacro:yumi_servo_gripper>
   <!--left gripper-->
-  <xacro:yumi_servo_gripper name="gripper_l" hardware_interface="$(arg prefix)" parent="yumi_link_7_l">
+  <xacro:yumi_servo_gripper name="gripper_l" hardware_interface="hardware_interface/EffortJointInterface" parent="yumi_link_7_l">
     <origin xyz="0 0 0.007" rpy="0 0 ${PI}" />
   </xacro:yumi_servo_gripper>
+  <!--yumi head-->
+  <joint name="head_to_yumi" type="fixed">
+  <parent link="yumi_base_link"/>
+  <child link="head_base_link"/>
+  <origin xyz="-0.12 0 0.62" rpy="0 0 0" />
+  </joint>
+  <link name="head_base_link"/>
+  <joint name="head_pan_joint" type="revolute">
+  <axis xyz="0 0 1" />
+  <limit lower="-${PI/4}" upper="${PI/4}" effort="1.0" velocity="3.14"/>
+  <parent link="head_base_link"/>
+  <child link="head_pan_link"/>
+  <origin xyz="0 0 0" rpy="0 0 0" />
+  </joint>
+  <link name="head_pan_link"/>
+  <joint name="head_tilt_joint" type="revolute">
+  <axis xyz="0 1 0" />
+  <limit lower="-${PI/4}" upper="${PI/4}" effort="1.0" velocity="3.14"/>
+  <parent link="head_pan_link"/>
+  <child link="head_tilt_link"/>
+  <origin xyz="0 0 0" rpy="0 0 0" />
+  </joint>
+  <link name="head_tilt_link">
+    <collision>
+      <origin xyz="0.05 0 0" rpy="0 0 0"/>
+      <geometry>
+    <box size="0.01 0.15 0.1"/>
+      </geometry>
+    </collision>
+    <visual>
+      <origin xyz="0.05 0 0" rpy="0 0 0"/>
+      <geometry>
+        <box size="0.01 0.15 0.1"/>
+      </geometry>
+      <material name="Grey" />
+    </visual>
+  </link>
+  <!-- Add ZR300 to yumi_base_link with the given transforms-->
+  <joint name="zr300_joint" type="fixed">
+	<origin xyz="-0.12 -0.03 0.23" rpy=" 0 0 0" />
+	<parent link="yumi_base_link" />
+	<child link="zr300_link" />
+  </joint>
+  <link name="zr300_link">
+	<visual>
+		<origin xyz="0.005 0.03 0" rpy="0 0 0" />
+		<geometry>
+			<box size="0.01 0.16 0.03"/>
+		</geometry>
+		<material name="black"/>
+	</visual>
+	<collision>
+		<origin xyz="0.005 0.03 0" rpy="0 0 0" />
+		<geometry>
+			<box size="0.01 0.16 0.03"/>
+		</geometry>
+		<material name="black"/>
+	</collision>
+  </link>
+  <!-- Add SR300 to yumi_base_link with the given transforms-->
+  <joint name="sr300_joint" type="fixed">
+	<origin xyz="0 0 0.28" rpy=" 0 0.98020367320510338076867830836025 0" />
+	<parent link="yumi_base_link" />
+	<child link="camera_link" />
+  </joint>
+  <link name="camera_link">
+	<visual>
+		<origin xyz="0 0 0" rpy="0 0 0" />
+		<geometry>
+			<box size="0.01 0.12 0.03"/>
+		</geometry>
+		<material name="black"/>
+	</visual>
+	<collision>
+		<origin xyz="0 0 0" rpy="0 0 0" />
+		<geometry>
+			<box size="0.01 0.12 0.03"/>
+		</geometry>
+		<material name="black"/>
+	</collision>
+  </link>
+  <!-- Add Leap Motion to yumi_base_link with the given transforms -->
+  <joint name="leap_joint" type="fixed">
+	<origin xyz="0.625 0 0.01" rpy="1.57079632679 0 1.57079632679" />
+	<parent link="yumi_base_link" />
+	<child link="leap" />
+  </joint>
+  <link name="leap">
+	<visual>
+		<origin xyz="0 0 0" rpy="0 0 0" />
+		<geometry>
+			<box size="0.08 0.01 0.03"/>
+		</geometry>
+		<material name="black"/>
+	</visual>
+	<collision>
+		<origin xyz="0 -0.01 0" rpy="0 0 0" />
+		<geometry>
+			<box size="0.08 0.01 0.03"/>
+		</geometry>
+		<material name="black"/>
+	</collision>
+  </link>
+  <!-- Yumi Table -->
+    <link name="yumi_base_link">
+    <collision>
+      <origin xyz="0.325 0 0" rpy="0 0 0"/>
+      <geometry>
+    <box size="0.65 0.65 0"/>
+      </geometry>
+    </collision>
+    <visual>
+      <origin xyz="0.325 0 0" rpy="0 0 0"/>
+      <geometry>
+        <box size="0.65 0.65 0"/>
+      </geometry>
+      <material name="Grey" />
+    </visual>
+    </link>
+    <xacro:property name="yumi_parent" value="world" />
+    <link name="world"/>
+    <joint name="world_joint" type="fixed">
+      <parent link="world"/>
+      <child link="yumi_base_link"/>
+      <origin xyz="0 0 0.1" rpy="0 0 0" />
+    </joint>
 </robot>

File: yumi_description/urdf/yumi.xacro (robot description, xacro)
@@ -2,20 +2,15 @@
 <robot name="yumi" xmlns:xacro="http://www.ros.org/wiki/xacro">
   <!-- Import all Gazebo-customization elements, including Gazebo colors -->
-  <xacro:include filename="$(find yumi_description)/urdf/yumi.gazebo.xacro" />
+  <xacro:include filename="$(find yumi_description)/urdf/Gazebo/yumi.gazebo.xacro" />
   <!-- Import Transmissions -->
   <xacro:include filename="$(find yumi_description)/urdf/yumi.transmission.xacro" />
-  <!-- Include Utilities -->
-  <xacro:include filename="$(find yumi_description)/urdf/utilities.xacro" />
   <!-- some constants -->
- <!-- <xacro:property name="safety_controller_k_pos" value="100" />
-  <xacro:property name="safety_controller_k_vel" value="2" /> -->
   <xacro:property name="joint_damping" value="0.5" />
   <xacro:property name="max_effort" value="300"/>
   <xacro:macro name="yumi" params="parent name hardware_interface *origin">
-    <!--joint between {parent} and body-->
-    <joint name="${parent}_joint" type="fixed">
-      <insert_block name="origin"/>
-      <parent link="${parent}"/>
+    <joint name="${name}_base_link_to_body" type="fixed">
+      <parent link="yumi_base_link"/>
       <child link="${name}_body"/>
+      <origin xyz="0 0 0" rpy="0 0 0"/>
     </joint>
     <link name="${name}_body">
@@ -49,8 +44,4 @@
       <limit lower="${-168.5 * PI / 180}" upper="${168.5 * PI / 180}"
              effort="${max_effort}" velocity="${180 * PI / 180}" />
-      <!--   <safety_controller soft_lower_limit="${-168 * M_PI / 180}"
-           soft_upper_limit="${168 * M_PI / 180}"
-           k_position="${safety_controller_k_pos}"
-           k_velocity="${safety_controller_k_vel}"/> -->
       <dynamics damping="${joint_damping}"/>
     </joint>
@@ -84,11 +75,7 @@
       <limit lower="${-143.5 * PI / 180}" upper="${43.5 * PI / 180}"
              effort="${max_effort}" velocity="${180 * PI / 180}" />
-      <!--   <safety_controller soft_lower_limit="${-168 * M_PI / 180}"
-           soft_upper_limit="${168 * M_PI / 180}"
-           k_position="${safety_controller_k_pos}"
-           k_velocity="${safety_controller_k_vel}"/> -->
-      <dynamics damping="${joint_damping}"/>
-    </joint>
-   <link name="${name}_link_2_r">
+      <dynamics damping="${joint_damping}"/>
+    </joint>
+    <link name="${name}_link_2_r">
       <inertial>
         <origin xyz="0 0 0" rpy="0 0 0"/>
@@ -111,19 +98,15 @@
       </collision>
     </link>
-   <!-- joint between link_2_r and link_3_r -->
-    <joint name="${name}_joint_7_r" type="revolute">
-      <parent link="${name}_link_2_r"/>
-      <child link="${name}_link_3_r"/>
-      <origin xyz="-0.03 0.17283 0.0" rpy="${-PI / 2} 0.0 0.0"/>
-      <axis xyz="0 0 1"/>
-      <limit lower="${-168.5 * PI / 180}" upper="${168.5 * PI / 180}"
-             effort="${max_effort}" velocity="${180 * PI / 180}" />
-      <!--   <safety_controller soft_lower_limit="${-168 * M_PI / 180}"
-           soft_upper_limit="${168 * M_PI / 180}"
-           k_position="${safety_controller_k_pos}"
-           k_velocity="${safety_controller_k_vel}"/> -->
-      <dynamics damping="${joint_damping}"/>
-    </joint>
-   <link name="${name}_link_3_r">
+     <!-- joint between link_2_r and link_3_r -->
+      <joint name="${name}_joint_7_r" type="revolute">
+        <parent link="${name}_link_2_r"/>
+        <child link="${name}_link_3_r"/>
+        <origin xyz="-0.03 0.17283 0.0" rpy="${-PI / 2} 0.0 0.0"/>
+        <axis xyz="0 0 1"/>
+        <limit lower="${-168.5 * PI / 180}" upper="${168.5 * PI / 180}"
+               effort="${max_effort}" velocity="${180 * PI / 180}" />
+        <dynamics damping="${joint_damping}"/>
+      </joint>
+    <link name="${name}_link_3_r">
       <inertial>
         <origin xyz="0 0 0" rpy="0 0 0"/>
@@ -146,5 +129,5 @@
       </collision>
     </link>
-   <!-- joint between link_3_r and link_4_r -->
+    <!-- joint between link_3_r and link_4_r -->
     <joint name="${name}_joint_3_r" type="revolute">
       <parent link="${name}_link_3_r"/>
@@ -154,11 +137,7 @@
       <limit lower="${-123.5 * PI / 180}" upper="${80 * PI / 180}"
              effort="${max_effort}" velocity="${180 * PI / 180}" />
-      <!--   <safety_controller soft_lower_limit="${-168 * M_PI / 180}"
-           soft_upper_limit="${168 * M_PI / 180}"
-           k_position="${safety_controller_k_pos}"
-           k_velocity="${safety_controller_k_vel}"/> -->
-      <dynamics damping="${joint_damping}"/>
-    </joint>
-   <link name="${name}_link_4_r">
+      <dynamics damping="${joint_damping}"/>
+    </joint>
+    <link name="${name}_link_4_r">
       <inertial>
         <origin xyz="0 0 0" rpy="0 0 0"/>
@@ -181,5 +160,5 @@
       </collision>
     </link>
-   <!-- joint between link_4_r and link_5_r -->
+    <!-- joint between link_4_r and link_5_r -->
     <joint name="${name}_joint_4_r" type="revolute">
       <parent link="${name}_link_4_r"/>
@@ -189,11 +168,7 @@
       <limit lower="${-290 * PI / 180}" upper="${290 * PI / 180}"
              effort="${max_effort}" velocity="${400 * PI / 180}" />
-      <!--   <safety_controller soft_lower_limit="${-168 * M_PI / 180}"
-           soft_upper_limit="${168 * M_PI / 180}"
-           k_position="${safety_controller_k_pos}"
-           k_velocity="${safety_controller_k_vel}"/> -->
-      <dynamics damping="${joint_damping}"/>
-    </joint>
-   <link name="${name}_link_5_r">
+      <dynamics damping="${joint_damping}"/>
+    </joint>
+    <link name="${name}_link_5_r">
       <inertial>
         <origin xyz="0 0 0" rpy="0 0 0"/>
@@ -216,5 +191,5 @@
       </collision>
     </link>
-   <!-- joint between link_5_r and link_6_r -->
+    <!-- joint between link_5_r and link_6_r -->
     <joint name="${name}_joint_5_r" type="revolute">
       <parent link="${name}_link_5_r"/>
@@ -224,11 +199,7 @@
       <limit lower="${-88 * PI / 180}" upper="${138 * PI / 180}"
              effort="${max_effort}" velocity="${400 * PI / 180}" />
-      <!--   <safety_controller soft_lower_limit="${-168 * M_PI / 180}"
-           soft_upper_limit="${168 * M_PI / 180}"
-           k_position="${safety_controller_k_pos}"
-           k_velocity="${safety_controller_k_vel}"/> -->
-      <dynamics damping="${joint_damping}"/>
-    </joint>
-   <link name="${name}_link_6_r">
+      <dynamics damping="${joint_damping}"/>
+    </joint>
+    <link name="${name}_link_6_r">
       <inertial>
         <origin xyz="0 0 0" rpy="0 0 0"/>
@@ -251,5 +222,5 @@
       </collision>
     </link>
-   <!-- joint between link_6_r and link_7_r -->
+    <!-- joint between link_6_r and link_7_r -->
     <joint name="${name}_joint_6_r" type="revolute">
       <parent link="${name}_link_6_r"/>
@@ -259,11 +230,7 @@
       <limit lower="${-229 * PI / 180}" upper="${229 * PI / 180}"
              effort="${max_effort}" velocity="${400 * PI / 180}" />
-      <!--   <safety_controller soft_lower_limit="${-168 * M_PI / 180}"
-           soft_upper_limit="${168 * M_PI / 180}"
-           k_position="${safety_controller_k_pos}"
-           k_velocity="${safety_controller_k_vel}"/> -->
-      <dynamics damping="${joint_damping}"/>
-    </joint>
-   <link name="${name}_link_7_r">
+      <dynamics damping="${joint_damping}"/>
+    </joint>
+    <link name="${name}_link_7_r">
       <inertial>
         <origin xyz="0 0 0" rpy="0 0 0"/>
@@ -286,6 +253,6 @@
       </collision>
     </link>
-   <!--///////////////////////////////////// LEFT ARM ////////////////////////////////  -->
-  <!-- joint between body and link_1_l -->
+    <!--///////////////////////////////////// LEFT ARM ////////////////////////////////  -->
+    <!-- joint between body and link_1_l -->
     <joint name="${name}_joint_1_l" type="revolute">
       <parent link="${name}_body"/>
@@ -295,11 +262,7 @@
       <limit lower="${-168.5 * PI / 180}" upper="${168.5 * PI / 180}"
              effort="${max_effort}" velocity="${180 * PI / 180}" />
-      <!--   <safety_controller soft_lower_limit="${-168 * M_PI / 180}"
-           soft_upper_limit="${168 * M_PI / 180}"
-           k_position="${safety_controller_k_pos}"
-           k_velocity="${safety_controller_k_vel}"/> -->
-      <dynamics damping="${joint_damping}"/>
-    </joint>
-   <link name="${name}_link_1_l">
+      <dynamics damping="${joint_damping}"/>
+    </joint>
+    <link name="${name}_link_1_l">
       <inertial>
         <origin xyz="0 -0.03 0.12" rpy="0 0 0"/>
@@ -322,5 +285,5 @@
       </collision>
     </link>
- <!-- joint between link_1_l and link_2_l -->
+    <!-- joint between link_1_l and link_2_l -->
     <joint name="${name}_joint_2_l" type="revolute">
       <parent link="${name}_link_1_l"/>
@@ -330,11 +293,7 @@
       <limit lower="${-143.5 * PI / 180}" upper="${43.5 * PI / 180}"
              effort="${max_effort}" velocity="${180 * PI / 180}" />
-      <!--   <safety_controller soft_lower_limit="${-168 * M_PI / 180}"
-           soft_upper_limit="${168 * M_PI / 180}"
-           k_position="${safety_controller_k_pos}"
-           k_velocity="${safety_controller_k_vel}"/> -->
-      <dynamics damping="${joint_damping}"/>
-    </joint>
-   <link name="${name}_link_2_l">
+      <dynamics damping="${joint_damping}"/>
+    </joint>
+    <link name="${name}_link_2_l">
       <inertial>
         <origin xyz="0 0 0" rpy="0 0 0"/>
@@ -357,5 +316,5 @@
       </collision>
     </link>
- <!-- joint between link_2_l and link_3_l -->
+    <!-- joint between link_2_l and link_3_l -->
     <joint name="${name}_joint_7_l" type="revolute">
       <parent link="${name}_link_2_l"/>
@@ -365,11 +324,7 @@
       <limit lower="${-168.5 * PI / 180}" upper="${168.5 * PI / 180}"
              effort="${max_effort}" velocity="${180 * PI / 180}" />
-      <!--   <safety_controller soft_lower_limit="${-168 * M_PI / 180}"
-           soft_upper_limit="${168 * M_PI / 180}"
-           k_position="${safety_controller_k_pos}"
-           k_velocity="${safety_controller_k_vel}"/> -->
-      <dynamics damping="${joint_damping}"/>
-    </joint>
-   <link name="${name}_link_3_l">
+      <dynamics damping="${joint_damping}"/>
+    </joint>
+    <link name="${name}_link_3_l">
       <inertial>
         <origin xyz="0 0 0" rpy="0 0 0"/>
@@ -392,5 +347,5 @@
       </collision>
     </link>
-   <!-- joint between link_3_l and link_4_l -->
+    <!-- joint between link_3_l and link_4_l -->
     <joint name="${name}_joint_3_l" type="revolute">
       <parent link="${name}_link_3_l"/>
@@ -400,11 +355,7 @@
       <limit lower="${-123.5 * PI / 180}" upper="${80 * PI / 180}"
              effort="${max_effort}" velocity="${180 * PI / 180}" />
-      <!--   <safety_controller soft_lower_limit="${-168 * M_PI / 180}"
-           soft_upper_limit="${168 * M_PI / 180}"
-           k_position="${safety_controller_k_pos}"
-           k_velocity="${safety_controller_k_vel}"/> -->
-      <dynamics damping="${joint_damping}"/>
-    </joint>
-   <link name="${name}_link_4_l">
+      <dynamics damping="${joint_damping}"/>
+    </joint>
+    <link name="${name}_link_4_l">
       <inertial>
         <origin xyz="0 0 0" rpy="0 0 0"/>
@@ -427,5 +378,5 @@
       </collision>
     </link>
-   <!-- joint between link_4_l and link_5_l -->
+    <!-- joint between link_4_l and link_5_l -->
     <joint name="${name}_joint_4_l" type="revolute">
       <parent link="${name}_link_4_l"/>
@@ -435,11 +386,7 @@
       <limit lower="${-290 * PI / 180}" upper="${290 * PI / 180}"
              effort="${max_effort}" velocity="${400 * PI / 180}" />
-      <!--   <safety_controller soft_lower_limit="${-168 * M_PI / 180}"
-           soft_upper_limit="${168 * M_PI / 180}"
-           k_position="${safety_controller_k_pos}"
-           k_velocity="${safety_controller_k_vel}"/> -->
-      <dynamics damping="${joint_damping}"/>
-    </joint>
-   <link name="${name}_link_5_l">
+      <dynamics damping="${joint_damping}"/>
+    </joint>
+    <link name="${name}_link_5_l">
       <inertial>
         <origin xyz="0 0 0" rpy="0 0 0"/>
@@ -462,5 +409,5 @@
       </collision>
     </link>
-   <!-- joint between link_5_l and link_6_l -->
+    <!-- joint between link_5_l and link_6_l -->
     <joint name="${name}_joint_5_l" type="revolute">
       <parent link="${name}_link_5_l"/>
@@ -470,11 +417,7 @@
       <limit lower="${-88 * PI / 180}" upper="${138 * PI / 180}"
              effort="${max_effort}" velocity="${400 * PI / 180}" />
-      <!--   <safety_controller soft_lower_limit="${-168 * M_PI / 180}"
-           soft_upper_limit="${168 * M_PI / 180}"
-           k_position="${safety_controller_k_pos}"
-           k_velocity="${safety_controller_k_vel}"/> -->
-      <dynamics damping="${joint_damping}"/>
-    </joint>
-   <link name="${name}_link_6_l">
+      <dynamics damping="${joint_damping}"/>
+    </joint>
+    <link name="${name}_link_6_l">
       <inertial>
         <origin xyz="0 0 0" rpy="0 0 0"/>
@@ -497,5 +440,5 @@
       </collision>
     </link>
-   <!-- joint between link_6_l and link_7_l -->
+    <!-- joint between link_6_l and link_7_l -->
     <joint name="${name}_joint_6_l" type="revolute">
       <parent link="${name}_link_6_l"/>
@@ -505,11 +448,7 @@
       <limit lower="${-229 * PI / 180}" upper="${229 * PI / 180}"
              effort="${max_effort}" velocity="${400 * PI / 180}" />
-      <!--   <safety_controller soft_lower_limit="${-168 * M_PI / 180}"
-           soft_upper_limit="${168 * M_PI / 180}"
-           k_position="${safety_controller_k_pos}"
-           k_velocity="${safety_controller_k_vel}"/> -->
-      <dynamics damping="${joint_damping}"/>
-    </joint>
-   <link name="${name}_link_7_l">
+      <dynamics damping="${joint_damping}"/>
+    </joint>
+    <link name="${name}_link_7_l">
       <inertial>
         <origin xyz="0 0 0" rpy="0 0 0"/>
