Commit message: user study preparation

File: yumi_description/urdf/yumi.urdf.xacro (robot description, xacro)
@@ -11,4 +11,6 @@
   <!-- Import Gazebo plugins -->
   <xacro:include filename="$(find yumi_description)/urdf/Gazebo/gazebo.urdf.xacro"/>
+  <!-- Import the D415 camera macro -->
+  <xacro:include filename="$(find realsense2_camera)/urdf/_d415.urdf.xacro"/>
   <!--yumi-->
   <xacro:yumi name="yumi" hardware_interface="hardware_interface/VelocityJointInterface" parent="${yumi_parent}" >
@@ -23,5 +25,5 @@
     <origin xyz="0 0 0.007" rpy="0 0 ${PI}" />
   </xacro:yumi_servo_gripper>
-  <!--yumi head-->
+  <!--yumi head>
   <joint name="head_to_yumi" type="fixed">
   <parent link="yumi_base_link"/>
@@ -59,6 +61,6 @@
       <material name="Grey" />
     </visual>
-  </link>
-  <!-- Add ZR300 to yumi_base_link with the given transforms-->
+  </link-->
+  <!-- Add ZR300 to yumi_base_link with the given transforms>
   <joint name="zr300_joint" type="fixed">
 	<origin xyz="-0.12 -0.03 0.23" rpy=" 0 0 0" />
@@ -81,8 +83,12 @@
 		<material name="black"/>
 	</collision>
-  </link>
-  <!-- Add SR300 to yumi_base_link with the given transforms-->
+  </link-->
+  <!--add D415 camera-->
+  <xacro:sensor_d415 parent="yumi_base_link">
+    <origin xyz="0.11 0 0.31" rpy="0 0 0" />
+  </xacro:sensor_d415>
+  <!-- Add SR300 to yumi_base_link with the given transforms>
   <joint name="sr300_joint" type="fixed">
-	<origin xyz="0 0 0.28" rpy=" 0 0.98020367320510338076867830836025 0" />
+	<origin xyz="0 0 0.28" rpy=" 0 0.80020367320510338076867830836025 0" />
 	<parent link="yumi_base_link" />
 	<child link="camera_link" />
@@ -103,8 +109,9 @@
 		<material name="black"/>
 	</collision>
-  </link>
+  </link-->
   <!-- Add Leap Motion to yumi_base_link with the given transforms -->
   <joint name="leap_joint" type="fixed">
-	<origin xyz="0.625 0 0.01" rpy="1.57079632679 0 1.57079632679" />
+	<!--origin xyz="0.625 0 0.01" rpy="1.57079632679 0 1.57079632679" /-->
+	<origin xyz="0.95 0 0.11" rpy="1.57079632679 0 1.57079632679" />
 	<parent link="yumi_base_link" />
 	<child link="leap" />
@@ -119,5 +126,5 @@
 	</visual>
 	<collision>
-		<origin xyz="0 -0.01 0" rpy="0 0 0" />
+		<origin xyz="0 0 0" rpy="0 0 0" />
 		<geometry>
 			<box size="0.08 0.01 0.03"/>
@@ -138,4 +145,51 @@
       <geometry>
         <box size="0.65 0.65 0"/>
+      </geometry>
+      <material name="Grey" />
+    </visual>
+    </link>
+  <!-- User Study Table -->
+    <joint name="user_study_joint" type="fixed">
+	<origin xyz="0 0 0" rpy="0 0 0" />
+	<parent link="yumi_base_link" />
+	<child link="user_study_link" />
+    </joint>
+    <link name="user_study_link">
+    <collision>
+      <origin xyz="0.65 0 0.1" rpy="0 0 0"/>
+      <geometry>
+    <box size="0.8 1.4 0"/>
+      </geometry>
+    </collision>
+    <collision>
+      <origin xyz="0.5 0 0.125" rpy="0 0 0"/>
+      <geometry>
+    <box size="0 1 0.05"/>
+      </geometry>
+    </collision>
+    <collision>
+      <origin xyz="0.25 0 0.1" rpy="0 0 0"/>
+      <geometry>
+    <box size="0 1 0.06"/>
+      </geometry>
+    </collision>
+    <visual>
+      <origin xyz="0.65 0 0.1" rpy="0 0 0"/>
+      <geometry>
+        <box size="0.8 1.4 0"/>
+      </geometry>
+      <material name="Grey" />
+    </visual>
+    <visual>
+      <origin xyz="0.5 0 0.125" rpy="0 0 0"/>
+      <geometry>
+        <box size="0 1 0.05"/>
+      </geometry>
+      <material name="Grey" />
+    </visual>
+    <visual>
+      <origin xyz="0.25 0 0.1" rpy="0 0 0"/>
+      <geometry>
+    <box size="0 1 0.06"/>
       </geometry>
       <material name="Grey" />
